File: cr2022012001-12-leds-board.kicad_pcb (KiCad board)
At the start: 2 copper layers, 79.7 x 67.8 mm, 38 parts, among them J1 USB_B_Micro, J2 Conn_01x04, SW1 SW_Push, U1 ATtiny85-20PU

Commit message: updated drawing
Parts:
- added D27: 3V6, Diode_THT:D_DO-41_SOD81_P7.62mm_Horizontal, B.Cu at (181.5, 82.5)
- added D28: 3V6, Diode_THT:D_DO-41_SOD81_P7.62mm_Horizontal, B.Cu at (181.5, 86.5)
- added J3: AVR-ISP-6, Connector_PinSocket_2.54mm:PinSocket_2x03_P2.54mm_Vertical, B.Cu at (192.5, 102.5)
- added R10: 100, Resistor_SMD:R_0603_1608Metric_Pad0.98x0.95mm_HandSolder, F.Cu at (196.9, 111.4)
- added R11: 100, Resistor_SMD:R_0603_1608Metric_Pad0.98x0.95mm_HandSolder, F.Cu at (206.9, 101.4)
- added R12: 1K, Resistor_SMD:R_0603_1608Metric_Pad0.98x0.95mm_HandSolder, F.Cu at (181.0, 74.9)
- added R13: 47, Resistor_SMD:R_0603_1608Metric_Pad0.98x0.95mm_HandSolder, F.Cu at (173.6, 78.0)
- added R14: 47, Resistor_SMD:R_0603_1608Metric_Pad0.98x0.95mm_HandSolder, F.Cu at (173.6, 73.5)
- added R8: 100, Resistor_SMD:R_0603_1608Metric_Pad0.98x0.95mm_HandSolder, F.Cu at (173.4, 101.1)
- added R9: 100, Resistor_SMD:R_0603_1608Metric_Pad0.98x0.95mm_HandSolder, F.Cu at (183.4, 111.1)
- added U2: ATtiny85-20SU, Package_SO:SOIJ-8_5.3x5.3mm_P1.27mm, B.Cu at (182.3, 94.6)
- BT1, D25, D26, J1, R5, R6, R7, SW1, U1: moved to B.Cu
- moved BT1 167.7 mm to (204.5, 83.5), turned to 45 degrees
- moved D11 146.5 mm to (222.0, 72.4), turned to 270 degrees
- moved R3 146.4 mm to (194.1, 108.6), turned to 315 degrees
- moved R4 142.5 mm to (204.1, 98.6), turned to 315 degrees
- moved D16 137.6 mm to (190.1, 71.5)
- moved D5 132.3 mm to (203.6, 108.4), turned to 225 degrees
- moved D10 132.1 mm to (223.6, 88.4), turned to 225 degrees
- moved D12 130.4 mm to (205.6, 63.0), turned to 180 degrees
- moved D6 129.1 mm to (213.6, 98.4), turned to 225 degrees
- moved R1 125.3 mm to (175.9, 98.6), turned to 225 degrees
- moved D4 113.8 mm to (190.0, 118.0)
- moved R2 109.4 mm to (185.9, 108.6), turned to 225 degrees
- moved R7 105.6 mm to (169.5, 73.5)
- moved R5 104.1 mm to (181.0, 79.0), turned to 90 degrees
- moved R6 100.9 mm to (177.1, 78.0), turned to 180 degrees
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Connections:
- J1 pad 4: Net-(J1-Pad4) -> (no net)
Routing:
- net Net-(D1-Pad1): track 0.00 -> 157.2 mm
- net Net-(D12-Pad1): track 0.00 -> 69.1 mm
- net Net-(D1-Pad2): track 0.00 -> 61.5 mm
- net Net-(D11-Pad1): track 0.00 -> 61.4 mm
- net Net-(J2-Pad4): track 0.00 -> 27.1 mm
- net Net-(J2-Pad1): track 0.00 -> 26.8 mm
- net Net-(J2-Pad3): track 0.00 -> 14.1 mm
- net Net-(J2-Pad2): track 0.00 -> 14.1 mm

Commit message: revNC
Parts:
- added G***: LOGO, CAROBOT_KiCad_Footprint:Logo_CAROBOT_Robot_5mm, B.Cu at (159.8, 54.3)
- added G***: LOGO, CAROBOT_KiCad_Footprint:Text_LOVE_9mm, F.Cu at (189.9, 79.4)
- added G***: LOGO, CAROBOT_KiCad_Footprint:Text_LOVE_12mm, F.Cu at (168.3, 65.6)
- added G***: LOGO, CAROBOT_KiCad_Footprint:Logo_CAROBOT_Robot_5mm, F.Cu at (195.2, 69.1)
- J1: footprint Connector_USB:USB_Micro-B_Molex-105017-0001 -> Connector_USB:USB_Micro-B_Amphenol_10118194_Horizontal
- R12, R13, R14: moved to B.Cu
- moved J2 44.4 mm to (152.0, 92.4), turned to 45 degrees
- moved D4 41.3 mm to (157.0, 93.1), turned to 315 degrees
- moved D22 40.0 mm to (154.1, 48.4), turned to 270 degrees
- moved D1 39.9 mm to (158.4, 91.7), turned to 45 degrees
- moved D19 38.8 mm to (156.3, 47.2), turned to 270 degrees
- moved D24 38.7 mm to (154.1, 76.7), turned to 270 degrees
- moved R9 38.0 mm to (157.1, 83.6), turned to 180 degrees
- moved D23 37.8 mm to (154.1, 62.6), turned to 270 degrees
- moved D21 36.9 mm to (156.3, 75.5), turned to 270 degrees
- moved D20 36.3 mm to (156.3, 61.3), turned to 270 degrees
- moved R8 35.6 mm to (157.1, 69.5), turned to 180 degrees
- moved R2 35.5 mm to (160.7, 83.6), turned to 180 degrees
- moved R10 35.3 mm to (166.5, 93.3), turned to 270 degrees
- moved D18 35.2 mm to (166.8, 38.1), turned to 225 degrees
- moved R3 33.6 mm to (166.5, 89.4), turned to 270 degrees
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Connections:
- J1 pad 4: (no net) -> Net-(J1-Pad4)
Routing:
- net VCC: track 0.00 -> 163.0 mm
- net Net-(D1-Pad2): track 61.5 -> 167.7 mm
- net Net-(D11-Pad1): track 61.4 -> 164.6 mm
- net GND: track 0.10 -> 85.1 mm
- net Net-(D12-Pad1): track 69.1 -> 144.6 mm
- net Net-(D26-Pad1): track 0.00 -> 58.6 mm
- net Net-(J2-Pad4): track 27.1 -> 83.7 mm
- net Net-(J2-Pad1): track 26.8 -> 79.0 mm
- net Net-(D25-Pad1): track 0.00 -> 51.5 mm
- net Net-(J2-Pad2): track 14.1 -> 50.0 mm
- net Net-(J2-Pad3): track 14.1 -> 44.3 mm
- net Net-(J3-Pad5): track 0.00 -> 28.9 mm
- net Net-(R13-Pad1): track 0.00 -> 24.6 mm
- net Net-(J1-Pad6): track 0.00 -> 12.0 mm
- net Net-(D1-Pad1): track 157.2 -> 165.2 mm
Other:
- board size 79.7 x 67.8 mm -> 68 x 68 mm
- board text added: "2022-01-21 JKL Rev-NC"
- board text added: "carobot.ca"
